File: schematic/sdr-trx/sdr-trx.kicad_pcb (KiCad board)
At the start: 2 copper layers, 645 parts, among them J1 PJ-036AH-SMT, J10 47346-0001, J2 SJ-3524-SMT-TR, J3 PJ1-022-SMT, J4 SJ-3524-SMT-TR-GR, J5 SJ-3524-SMT-TR-BE, J6 SJ-3524-SMT-TR-PI, J7 CON-SMA-EDGE, J8 TSM-103-02, J9 DM3D-SF, K1 AGQ200A12, K2 AGQ200A12, K3 AGQ200A12, K4 AGQ200A12, K5 AGQ200A12, K6 AGQ200A12, K7 AGQ200A12, Q1 BSS138P, Q10 BSS138P, Q11 BSS138P, Q12 BSS138P, Q13 BSS138P, Q14 Si4909DY, Q15 BCP52, Q16 2SB1198K, Q17 BSS138P, Q18 DMP3099L, Q19 BSS138P, Q2 BSS138P, Q20 2SC2412K, Q21 DMP3099L, Q22 Si4909DY, Q23 2SC2412K, Q24 2SB1198K, Q25 2SC2412K, Q26 2SB1198K, Q27 BSS138P, Q28 BSS138P, Q29 BSS138P, Q3 MMBT2222A, Q4 BFU520W, Q5 DZT2222A, Q6 PD85004, Q7 PD85004, Q8 BSS138P, Q9 Si4909DY, SW1 EVQP7A, SW2 EVQP7A, T1 BN43-202, T2 BN43-202, U1 Si5351A-B-GT, U10 SN74HC126P, U11 SN74CBT3253C, U12 SN74CBT3305C, U13 SN74CBT3253C, U14 SN74CBT3305C, U15 AD5243BRMZ, U16 ULN2003V12T16-13, U17 LTC5507, U18 LTC5507, U19 TCA0372BDW, U2 PO74G74A, U20 WM8731, U21 74HC4066PW, U22 74HC4066PW, U23 SN74HC00P, U24 STM32F413RHTx, U25 M24C64-RDW, U26 NUP4202, U27 NUP4202, U28 SN74HC595P, U29 LF50ABPT, U3 AD8604, U30 LF50ABPT, U31 LF50ABPT, U32 LF50ABPT, U33 LF50ABPT, U34 LF33CPT, U35 LF33CPT, U36 LF33CPT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

Commit message: Route PCB.
Parts:
- BT2, BT3, BT4: moved to B.Cu
- D1, D6, D7, D8: footprint Package_TO_SOT_SMD:SOT-23_Handsoldering -> Diode_SMD:D_SOT-23_ANK
- Y1: footprint Crystal:Crystal_SMD_HC49-SD_HandSoldering -> Crystal:Crystal_SMD_HC49-SD
- moved C2 455.2 mm to (116.5, 82.2)
- moved R1 453.7 mm to (113.0, 86.2), turned to 270 degrees
- moved J6 453.0 mm to (39.5, 60.7), turned to 90 degrees
- moved R2 450.4 mm to (121.0, 86.2), turned to 90 degrees
- moved C1 448.4 mm to (116.5, 80.2)
- moved R3 444.9 mm to (122.0, 83.2)
- moved X1 444.2 mm to (117.0, 86.2)
- moved C5 444.1 mm to (130.0, 84.7)
- moved C47 440.5 mm to (129.0, 142.7), turned to 270 degrees
- moved J5 439.9 mm to (39.5, 48.7), turned to 90 degrees
- moved C44 439.8 mm to (127.0, 142.7), turned to 270 degrees
- moved C6 439.7 mm to (130.0, 82.7)
- moved C3 439.7 mm to (125.0, 86.2), turned to 90 degrees
- moved J3 439.6 mm to (42.0, 26.7), turned to 270 degrees
- moved C4 439.4 mm to (129.5, 90.7), turned to 180 degrees
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Connections:
- C236 pad 2: Net-(C236-Pad2) -> GND
- R96 pad 2: +3.3VA -> +3.3V
- R97 pad 2: Net-(C236-Pad2) -> GND
- TR3 pad 1: Net-(C142-Pad1) -> Net-(C143-Pad1)
- TR3 pad 3: Net-(C143-Pad1) -> Net-(C142-Pad1)
- TR3 pad 4: GND -> Net-(C136-Pad2)
- TR3 pad 6: Net-(C136-Pad2) -> GND
- U26 pad 4: /MCU/USB-DM -> (no net)
- U26 pad 6: (no net) -> /MCU/USB-DM
- U3 pad 13: Net-(R13-Pad2) -> Net-(R11-Pad1)
- U3 pad 14: Net-(R15-Pad2) -> Net-(R11-Pad2)
- U3 pad 8: Net-(R11-Pad2) -> Net-(R15-Pad2)
- U3 pad 9: Net-(R11-Pad1) -> Net-(R13-Pad2)
Routing:
- net /BPF/TX-EN: track 0.00 -> 483.3 mm, vias 0 -> 13
- net /BPF/RX-EN: track 0.00 -> 466.0 mm, vias 0 -> 8
- net /MCU/PTT-BTN: track 0.00 -> 441.5 mm, vias 0 -> 7
- net +3.3VA: track 0.00 -> 409.5 mm, vias 0 -> 15
- net +12V: track 0.00 -> 355.3 mm, vias 0 -> 7
- net /MCU/FWD: track 0.00 -> 325.3 mm, vias 0 -> 2
- net /MCU/REV: track 0.00 -> 317.8 mm, vias 0 -> 2
- net +5.0V-USB: track 0.00 -> 273.8 mm, vias 0 -> 4
- net +5.0V-TX: track 0.00 -> 271.1 mm, vias 0 -> 13
- net /BPF/BAND0: track 0.00 -> 265.8 mm, vias 0 -> 6
- net +5.0V-RX: track 0.00 -> 264.9 mm, vias 0 -> 10
- net GND: track 0.00 -> 258.5 mm, vias 0 -> 475
- net /MCU/PWR-BTN: track 0.00 -> 252.4 mm, vias 0 -> 7
- net /BPF/BAND1: track 0.00 -> 246.4 mm, vias 0 -> 5
- net Net-(C214-Pad2): track 0.00 -> 207.9 mm, vias 0 -> 2
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- added copper zone on F.Cu, net +12V
- added copper zone on F.Cu, net +12V-RF
- added copper zone on In2.Cu, net +12V-RF
- added copper zone on F.Cu, net +12V-TX
- added copper zone on In2.Cu, net +12V-TX
- added copper zone on In2.Cu, net +3.3V
- added copper zone on In2.Cu, net +3.3V-RF
- added copper zone on In2.Cu, net +3.3VA
- added copper zone on In2.Cu, net +5.0V-RF
- added copper zone on In2.Cu, net +5.0V-RX
- added copper zone on F.Cu, net +5.0V-TX
- added copper zone on In2.Cu, net +5.0V-TX
- added copper zone on F.Cu, net /MCU/BAT
- added copper zone on In2.Cu, net /MCU/BAT
- added copper zone on F.Cu, net /PSU/VIN
- added copper zone on B.Cu, net GND
- added copper zone on F.Cu, net GND
- added copper zone on In1.Cu, net GND
- added copper zone on F.Cu, net Net-(C134-Pad2)
- added copper zone on F.Cu, net Net-(C148-Pad2)
- added copper zone on F.Cu, net Net-(C149-Pad2)
- added copper zone on F.Cu, net Net-(C63-Pad2)
- added copper zone on F.Cu, net Net-(D5-Pad2)
- added copper zone on F.Cu, net Net-(F1-Pad2)
- added copper zone on F.Cu, net Net-(Q21-Pad3)
Other:
- board outline added: 238.4 x 144.7 mm
- copper layers 2 -> 4
- net class Default: clearance 0.2 -> 0.15; trace_width 0.25 -> 0.3; via_dia 0.8 -> 0.7
- rule pad_to_mask_clearance: 0.051 -> 0.0762
- rule solder_mask_min_width: 0.25 -> 0.254
- rule trace_clearance: 0.2 -> 0.15
- rule trace_min: 0.2 -> 0.3
- rule via_min_drill: 0.3 -> 0.4
- rule via_min_size: 0.4 -> 0.7
- board text added: "Button caps: BTNK0390 https://www.ckswitches.com/media/1457/ksa_ksl.pdf"

Commit message: Generate PCB documentation.
Parts:
- added REF**: OSHW-Logo_19x20mm_SilkScreen, Symbol:OSHW-Logo_19x20mm_SilkScreen, F.Cu at (83.0, 58.2)
Routing:
- net GND: vias 475 -> 478
Other:
- board text added: "06-2020"
- board text added: "SDR-TRX v1.0"
