File: schematic/sdr-trx/sdr-trx.kicad_pcb (KiCad board)
At the start: 4 copper layers, 238.4 x 144.7 mm, 646 parts, among them J1 PJ-036AH-SMT, J10 47346-0001, J2 SJ-3524-SMT-TR, J3 PJ1-022-SMT, J4 SJ-3524-SMT-TR-GR, J5 SJ-3524-SMT-TR-BE, J6 SJ-3524-SMT-TR-PI, J7 CON-SMA-EDGE, J8 TSM-103-02, J9 DM3D-SF, K1 AGQ200A12, K2 AGQ200A12, K3 AGQ200A12, K4 AGQ200A12, K5 AGQ200A12, K6 AGQ200A12, K7 AGQ200A12, Q1 BSS138P, Q10 BSS138P, Q11 BSS138P, Q12 BSS138P, Q13 BSS138P, Q14 Si4909DY, Q15 BCP52, Q16 2SB1198K, Q17 BSS138P, Q18 DMP3099L, Q19 BSS138P, Q2 BSS138P, Q20 2SC2412K, Q21 DMP3099L, Q22 Si4909DY, Q23 2SC2412K, Q24 2SB1198K, Q25 2SC2412K, Q26 2SB1198K, Q27 BSS138P, Q28 BSS138P, Q29 BSS138P, Q3 MMBT2222A, Q4 BFU520W, Q5 DZT2222A, Q6 PD85004, Q7 PD85004, Q8 BSS138P, Q9 Si4909DY, SW1 EVQP7A, SW2 EVQP7A, T1 BN43-202, T2 BN43-202, U1 Si5351A-B-GT, U10 SN74HC126P, U11 SN74CBT3253C, U12 SN74CBT3305C, U13 SN74CBT3253C, U14 SN74CBT3305C, U15 AD5243BRMZ, U16 ULN2003V12T16-13, U17 LTC5507, U18 LTC5507, U19 TCA0372BDW, U2 PO74G74A, U20 WM8731, U21 74HC4066PW, U22 74HC4066PW, U23 SN74HC00P, U24 STM32F413RHTx, U25 M24C64-RDW, U26 NUP4202, U27 NUP4202, U28 SN74HC595P, U29 LF50ABPT, U3 AD8604, U30 LF50ABPT, U31 LF50ABPT, U32 LF50ABPT, U33 LF50ABPT, U34 LF33CPT, U35 LF33CPT, U36 LF33CPT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

Commit message: Extend specification (Add Digikey partnumbers). Minor schematic changes.
Parts:
- C194: value 1nF -> 1.0nF
- C34, C35, C36, C37: value 8.2nF 1% -> N/A
- D1: value BZX84C4V7 -> BZX84-C4V7
- R21, R22: value 100R 1% -> 100R
- U4: value AD8604 -> AD8618
Changed lines of the file:
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@@
       (effects (font (size 1 1) (thickness 0.15)))
     )
-    (fp_text value BZX84C4V7 (at 0 2.5 90) (layer F.Fab)
+    (fp_text value BZX84-C4V7 (at 0 2.5 90) (layer F.Fab)
       (effects (font (size 1 1) (thickness 0.15)))
     )
@@
       (effects (font (size 1 1) (thickness 0.15)))
     )
-    (fp_text value AD8604 (at 0 5.28) (layer F.Fab)
+    (fp_text value AD8618 (at 0 5.28) (layer F.Fab)
       (effects (font (size 1 1) (thickness 0.15)))
     )
@@
       (effects (font (size 1 1) (thickness 0.15)))
     )
-    (fp_text value "100R 1%" (at 0 1.65 90) (layer F.Fab)
+    (fp_text value 100R (at 0 1.65 90) (layer F.Fab)
       (effects (font (size 1 1) (thickness 0.15)))
     )
@@
       (effects (font (size 1 1) (thickness 0.15)))
     )
-    (fp_text value "100R 1%" (at 0 1.65) (layer F.Fab)
+    (fp_text value 100R (at 0 1.65) (layer F.Fab)
       (effects (font (size 1 1) (thickness 0.15)))
     )
@@
       (effects (font (size 1 1) (thickness 0.15)))
     )
-    (fp_text value 1nF (at 0 1.65 90) (layer F.Fab)
+    (fp_text value 1.0nF (at 0 1.65 90) (layer F.Fab)
       (effects (font (size 1 1) (thickness 0.15)))
     )
@@
       (effects (font (size 1 1) (thickness 0.15)))
     )
-    (fp_text value "8.2nF 1%" (at 0 1.65 90) (layer F.Fab)
+    (fp_text value N/A (at 0 1.65 90) (layer F.Fab)
       (effects (font (size 1 1) (thickness 0.15)))
     )
@@
       (effects (font (size 1 1) (thickness 0.15)))
     )
-    (fp_text value "8.2nF 1%" (at 0 1.65 90) (layer F.Fab)
+    (fp_text value N/A (at 0 1.65 90) (layer F.Fab)
       (effects (font (size 1 1) (thickness 0.15)))
     )
@@
       (effects (font (size 1 1) (thickness 0.15)))
     )
-    (fp_text value "8.2nF 1%" (at 0 1.65 90) (layer F.Fab)
+    (fp_text value N/A (at 0 1.65 90) (layer F.Fab)
       (effects (font (size 1 1) (thickness 0.15)))
     )
@@
       (effects (font (size 1 1) (thickness 0.15)))
     )
-    (fp_text value "8.2nF 1%" (at 0 1.65 90) (layer F.Fab)
+    (fp_text value N/A (at 0 1.65 90) (layer F.Fab)
       (effects (font (size 1 1) (thickness 0.15)))
     )
